Commit message: feat: add collision-safe MuJoCo workflow

File: ubuntu/ros_jazzy/exo_identify/urdf/exo.SLDASM/urdf/装配体.SLDASM.urdf (robot description, URDF)
Before this commit: robot 装配体.SLDASM, 8 links, 7 joints
Joints:
- joint joint1: axis 0 0 -1 -> 0 0 1
- joint joint2: axis 0 0 -1 -> 0 0 1
- joint joint3: axis 0 0 -1 -> 0 0 1
- joint joint4: axis 0 0 -1 -> 0 0 1
- joint joint5: axis 0 0 -1 -> 0 0 1
- joint joint6: axis 0 0 -1 -> 0 0 1
- joint joint7: axis 0 0 -1 -> 0 0 1
